Commit message: feat: add noncyclic 12dof GMR clip training

File: resources/robots/x1/urdf/X1_12DOF.urdf (robot description, URDF)
Before this commit: robot x1, 60 links, 59 joints
Links:
- link left_knee_pitch_link: mass 1.51225735 -> 1.5122608
- link right_knee_pitch_link: mass 1.51225735 -> 1.50954
